File: f103.kicad_pcb (KiCad board)
At the start: 2 copper layers, 337.2 x 122.6 mm, 211 parts, among them J1 Conn_01x04_Female, J2 Conn_01x01_Male, J3 Conn_01x01_Male, J4 Conn_01x01_Male, Q1 2N7002, SW1 Rotary_Encoder_Switch, U1 STM32F103CBTx, U2 XC6206P332MR, U3 SRV05-4, Y1 8MHz

Commit message: Add Production Files, Submit for review
Other:
- board text added: "1.75u"
- board text added: "2.75u"
Changed lines of the file:
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@@
   (general
     (thickness 1.6)
-    (drawings 2176)
+    (drawings 2178)
     (tracks 2419)
     (zones 0)
@@
   )
   (setup
-    (last_trace_width 0.254)
+    (last_trace_width 0.508)
     (user_trace_width 0.254)
     (user_trace_width 0.29972)
@@
     (tags resistor)
     (attr smd)
-    (fp_text reference R1 (at -2.552798 -0.009331 90) (layer B.SilkS)
+    (fp_text reference R1 (at -0.9652 1.6764 180) (layer B.SilkS)
       (effects (font (size 1 1) (thickness 0.15)) (justify mirror))
     )
@@
     (pad 1 np_thru_hole circle (at 0 0) (size 5 5) (drill 5) (layers *.Cu *.Mask))
   )
+  (gr_text 1.75u (at 294.894 108.966) (layer F.SilkS)
+    (effects (font (size 2 2) (thickness 0.3)))
+  )
+  (gr_text 2.75u (at 312.166 113.538) (layer F.SilkS)
+    (effects (font (size 2 2) (thickness 0.3)))
+  )
   (gr_text VBUS (at 160.984499 40.568146) (layer B.SilkS)
     (effects (font (size 1 1) (thickness 0.15)) (justify mirror))
   )
-  (gr_text Center (at 45.305669 88.726547) (layer F.SilkS)
-    (effects (font (size 1 1) (thickness 0.15)))
+  (gr_text Center (at 46.736 91.313) (layer F.SilkS)
+    (effects (font (size 2 2) (thickness 0.3)))
   )
-  (gr_text Stepped (at 27.843521 88.726546) (layer F.SilkS)
-    (effects (font (size 1 1) (thickness 0.15)))
+  (gr_text Stepped (at 26.162 91.186) (layer F.SilkS)
+    (effects (font (size 2 2) (thickness 0.3)))
   )
   (gr_text JLCJLCJLCJLC (at 164.210299 102.442547 45) (layer B.SilkS)
     (effects (font (size 0.85 0.85) (thickness 0.16)) (justify mirror))
   )
-  (gr_text 1u (at 152.653299 146.384546 -12) (layer F.SilkS)
-    (effects (font (size 1 1) (thickness 0.15)))
+  (gr_text 1u (at 155.829 145.161 -12) (layer F.SilkS)
+    (effects (font (size 2 2) (thickness 0.3)))
   )
-  (gr_text 1.25u (at 146.557299 145.114547 -12) (layer F.SilkS)
-    (effects (font (size 1 1) (thickness 0.15)))
+  (gr_text 1.25u (at 142.621 142.367 -12) (layer F.SilkS)
+    (effects (font (size 2 2) (thickness 0.3)))
   )
-  (gr_text 2.00u (at 115.569299 138.510547 -12) (layer F.SilkS)
-    (effects (font (size 1 1) (thickness 0.15)))
+  (gr_text 2.00u (at 112.649 134.239 -12) (layer F.SilkS)
+    (effects (font (size 2 2) (thickness 0.3)))
   )
-  (gr_text 2.25u (at 123.8243 140.288547 -12) (layer F.SilkS)
-    (effects (font (size 1 1) (thickness 0.15)))
+  (gr_text 2.25u (at 128.27 137.541 -12) (layer F.SilkS)
+    (effects (font (size 2 2) (thickness 0.3)))
   )
   (gr_text SWCLK (at 173.265399 123.906547) (layer B.SilkS)

Commit message: DRC I
Parts:
- removed J1: Conn_01x04_Female, Connector_PinHeader_2.54mm:PinHeader_1x04_P2.54mm_Vertical
Routing:
- net GND: track 191.3 -> 186.3 mm, vias 27 -> 28
- net VBUS: track 21.8 -> 17.2 mm, vias 1 -> 2
Changed lines of the file:
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@@
     (thickness 1.6)
     (drawings 2178)
-    (tracks 2419)
+    (tracks 2418)
     (zones 0)
-    (modules 211)
+    (modules 210)
     (nets 189)
   )
@@
   )
   (setup
-    (last_trace_width 0.508)
+    (last_trace_width 0.29972)
     (user_trace_width 0.254)
     (user_trace_width 0.29972)
@@
     (fp_arc (start -8 2.5) (end -8 3.5) (angle 90) (layer B.Cu) (width 0.5))
   )
-  (module Connector_PinHeader_2.54mm:PinHeader_1x04_P2.54mm_Vertical (layer B.Cu)
-    (at 168.241182 40.339546 270)
-    (descr "Through hole straight pin header, 1x04, 2.54mm pitch, single row")
-    (tags "Through hole pin header THT 1x04 2.54mm single row")
-    (fp_text reference J1 (at 1.778 3.751483) (layer B.Fab)
-      (effects (font (size 1 1) (thickness 0.15)) (justify mirror))
-    )
-    (fp_text value Conn_01x04_Female (at -2.2352 -14.053917) (layer B.Fab)
-      (effects (font (size 1 1) (thickness 0.15)) (justify mirror))
-    )
-    (fp_text user %R (at 0 0 180) (layer B.Fab)
-      (effects (font (size 1 1) (thickness 0.15)) (justify mirror))
-    )
-    (fp_line (start 1.8 5.61) (end -1.8 5.61) (layer B.CrtYd) (width 0.05))
-    (fp_line (start 1.8 -5.59) (end 1.8 5.61) (layer B.CrtYd) (width 0.05))
-    (fp_line (start -1.8 -5.59) (end 1.8 -5.59) (layer B.CrtYd) (width 0.05))
-    (fp_line (start -1.8 5.61) (end -1.8 -5.59) (layer B.CrtYd) (width 0.05))
-    (fp_line (start -1.33 5.14) (end 0 5.14) (layer B.SilkS) (width 0.12))
-    (fp_line (start -1.33 3.81) (end -1.33 5.14) (layer B.SilkS) (width 0.12))
-    (fp_line (start -1.33 2.54) (end 1.33 2.54) (layer B.SilkS) (width 0.12))
-    (fp_line (start 1.33 2.54) (end 1.33 -5.14) (layer B.SilkS) (width 0.12))
-    (fp_line (start -1.33 2.54) (end -1.33 -5.14) (layer B.SilkS) (width 0.12))
-    (fp_line (start -1.33 -5.14) (end 1.33 -5.14) (layer B.SilkS) (width 0.12))
-    (fp_line (start -1.27 4.445) (end -0.635 5.08) (layer B.Fab) (width 0.1))
-    (fp_line (start -1.27 -5.08) (end -1.27 4.445) (layer B.Fab) (width 0.1))
-    (fp_line (start 1.27 -5.08) (end -1.27 -5.08) (layer B.Fab) (width 0.1))
-    (fp_line (start 1.27 5.08) (end 1.27 -5.08) (layer B.Fab) (width 0.1))
-    (fp_line (start -0.635 5.08) (end 1.27 5.08) (layer B.Fab) (width 0.1))
-    (pad 4 thru_hole oval (at 0 -3.81 270) (size 1.7 1.7) (drill 1) (layers *.Cu *.Mask)
-      (net 1 GND))
-    (pad 3 thru_hole oval (at 0 -1.27 270) (size 1.7 1.7) (drill 1) (layers *.Cu *.Mask)
-      (net 11 D+))
-    (pad 2 thru_hole oval (at 0 1.27 270) (size 1.7 1.7) (drill 1) (layers *.Cu *.Mask)
-      (net 12 D-))
-    (pad 1 thru_hole rect (at 0 3.81 270) (size 1.7 1.7) (drill 1) (layers *.Cu *.Mask)
-      (net 184 VBUS))
-  )
   (module LED_THT:LED_D3.0mm (layer F.Cu)
     (at 0.712252 131.59891)
@@
   (segment (start 166.356763 99.852047) (end 168.338264 97.870547) (width 0.29972) (layer B.Cu) (net 1))
   (segment (start 166.292797 99.852048) (end 166.356763 99.852047) (width 0.29972) (layer B.Cu) (net 1))
-  (segment (start 172.733668 48.177115) (end 172.733668 41.036378) (width 0.508) (layer B.Cu) (net 1))
   (segment (start 172.051182 40.353891) (end 172.051182 40.339547) (width 0.508) (layer B.Cu) (net 1))
   (segment (start 172.733668 41.036378) (end 172.051182 40.353891) (width 0.508) (layer B.Cu) (net 1))
@@
   (segment (start 168.241183 45.223818) (end 168.241182 46.40243) (width 0.508) (layer B.Cu) (net 1))
   (segment (start 168.241182 46.40243) (end 168.248899 46.410146) (width 0.508) (layer B.Cu) (net 1))
-  (segment (start 172.051182 40.382629) (end 172.051182 40.339547) (width 0.508) (layer F.Cu) (net 1))
-  (segment (start 172.733668 41.065116) (end 172.051182 40.382629) (width 0.508) (layer F.Cu) (net 1))
-  (segment (start 172.733668 44.135177) (end 172.733668 41.065116) (width 0.508) (layer F.Cu) (net 1))
-  (segment (start 168.248899 46.410146) (end 170.458699 46.410147) (width 0.508) (layer F.Cu) (net 1))
-  (segment (start 170.458699 46.410147) (end 172.733668 44.135177) (width 0.508) (layer F.Cu) (net 1))
   (via (at 165.2524 46.3804) (size 1.016) (drill 0.762) (layers F.Cu B.Cu) (net 1))
   (via (at 20.7772 88.4174) (size 1.016) (drill 0.762) (layers F.Cu B.Cu) (net 1))
@@
   (via (at 166.4462 87.503) (size 0.8) (drill 0.4) (layers F.Cu B.Cu) (net 1))
   (via (at 157.0736 91.2114) (size 0.8) (drill 0.4) (layers F.Cu B.Cu) (net 1))
+  (via (at 172.733668 46.368668) (size 1.016) (drill 0.762) (layers F.Cu B.Cu) (net 1))
+  (segment (start 172.69219 46.410146) (end 172.733668 46.368668) (width 0.508) (layer F.Cu) (net 1))
+  (segment (start 168.248899 46.410146) (end 172.69219 46.410146) (width 0.508) (layer F.Cu) (net 1))
+  (segment (start 172.733668 48.177115) (end 172.733668 46.368668) (width 0.508) (layer B.Cu) (net 1))
+  (segment (start 172.733668 46.368668) (end 172.733668 41.036378) (width 0.508) (layer B.Cu) (net 1))
   (segment (start 168.587146 104.851915) (end 170.156343 106.421114) (width 0.29972) (layer B.Cu) (net 6))
   (segment (start 168.19525 104.851914) (end 168.587146 104.851915) (width 0.29972) (layer B.Cu) (net 6))
@@
   (segment (start 174.297099 44.530546) (end 174.246299 44.581346) (width 0.508) (layer B.Cu) (net 184))
   (segment (start 175.640299 44.530546) (end 174.297099 44.530546) (width 0.508) (layer B.Cu) (net 184))
-  (segment (start 167.042251 37.728477) (end 164.431182 40.339546) (width 0.508) (layer B.Cu) (net 184))
-  (segment (start 167.042251 37.06036) (end 167.042251 37.728477) (width 0.508) (layer B.Cu) (net 184))
-  (segment (start 165.751982 39.018747) (end 164.431182 40.339546) (width 0.508) (layer F.Cu) (net 184))
-  (segment (start 173.049499 39.018747) (end 165.751982 39.018747) (width 0.508) (layer F.Cu) (net 184))
-  (segment (start 175.640299 44.530546) (end 175.640299 41.609546) (width 0.508) (layer F.Cu) (net 184))
-  (segment (start 175.640299 41.609546) (end 173.049499 39.018747) (width 0.508) (layer F.Cu) (net 184))
+  (via (at 166.116 39.751) (size 1.016) (drill 0.762) (layers F.Cu B.Cu) (net 184))
+  (segment (start 167.042251 37.06036) (end 167.042251 38.824749) (width 0.508) (layer B.Cu) (net 184))
+  (segment (start 167.042251 38.824749) (end 166.116 39.751) (width 0.508) (layer B.Cu) (net 184))
+  (segment (start 166.116 39.751) (end 166.116 41.402) (width 0.508) (layer F.Cu) (net 184))
+  (segment (start 169.244546 44.530546) (end 175.640299 44.530546) (width 0.508) (layer F.Cu) (net 184))
+  (segment (start 166.116 41.402) (end 169.244546 44.530546) (width 0.508) (layer F.Cu) (net 184))
   (via (at 163.041899 87.710546) (size 0.8) (drill 0.4) (layers F.Cu B.Cu) (net 187))
   (segment (start 163.78275 97.93942) (end 163.78275 88.451397) (width 0.29972) (layer B.Cu) (net 187))

Commit message: DRC II
update silks and ground planes
Routing:
- net GND: vias 28 -> 31
Other:
- board text removed: "1.75u"
- board text removed: "2.75u"
- board text removed: "Center"
- board text removed: "Stepped"
- board text removed: "VBUS"
Changed lines of the file:
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@@
   (general
     (thickness 1.6)
-    (drawings 2178)
-    (tracks 2418)
+    (drawings 2173)
+    (tracks 2422)
     (zones 0)
     (modules 210)
@@
     (pad 1 np_thru_hole circle (at 0 0) (size 5 5) (drill 5) (layers *.Cu *.Mask))
   )
-  (gr_text 1.75u (at 294.894 108.966) (layer F.SilkS)
-    (effects (font (size 2 2) (thickness 0.3)))
-  )
-  (gr_text 2.75u (at 312.166 113.538) (layer F.SilkS)
-    (effects (font (size 2 2) (thickness 0.3)))
-  )
-  (gr_text VBUS (at 160.984499 40.568146) (layer B.SilkS)
-    (effects (font (size 1 1) (thickness 0.15)) (justify mirror))
-  )
-  (gr_text Center (at 46.736 91.313) (layer F.SilkS)
-    (effects (font (size 2 2) (thickness 0.3)))
-  )
-  (gr_text Stepped (at 26.162 91.186) (layer F.SilkS)
-    (effects (font (size 2 2) (thickness 0.3)))
-  )
   (gr_text JLCJLCJLCJLC (at 164.210299 102.442547 45) (layer B.SilkS)
     (effects (font (size 0.85 0.85) (thickness 0.16)) (justify mirror))
   )
-  (gr_text 1u (at 155.829 145.161 -12) (layer F.SilkS)
-    (effects (font (size 2 2) (thickness 0.3)))
+  (gr_text 1u (at 155.575 142.621 -12) (layer B.SilkS)
+    (effects (font (size 1.5 1.5) (thickness 0.2)) (justify mirror))
   )
-  (gr_text 1.25u (at 142.621 142.367 -12) (layer F.SilkS)
-    (effects (font (size 2 2) (thickness 0.3)))
+  (gr_text 1.25u (at 145.542 140.843 -12) (layer B.SilkS)
+    (effects (font (size 1.5 1.5) (thickness 0.2)) (justify mirror))
   )
-  (gr_text 2.00u (at 112.649 134.239 -12) (layer F.SilkS)
-    (effects (font (size 2 2) (thickness 0.3)))
+  (gr_text 2.00u (at 114.3 134.239 -12) (layer B.SilkS)
+    (effects (font (size 1.5 1.5) (thickness 0.2)) (justify mirror))
   )
-  (gr_text 2.25u (at 128.27 137.541 -12) (layer F.SilkS)
-    (effects (font (size 2 2) (thickness 0.3)))
+  (gr_text 2.25u (at 126.492 136.779 -12) (layer B.SilkS)
+    (effects (font (size 1.5 1.5) (thickness 0.2)) (justify mirror))
   )
   (gr_text SWCLK (at 173.265399 123.906547) (layer B.SilkS)
@@
   (segment (start 172.733668 48.177115) (end 172.733668 46.368668) (width 0.508) (layer B.Cu) (net 1))
   (segment (start 172.733668 46.368668) (end 172.733668 41.036378) (width 0.508) (layer B.Cu) (net 1))
+  (via (at 147.32 140.208) (size 0.8) (drill 0.4) (layers F.Cu B.Cu) (net 1))
+  (via (at 296.545 107.95) (size 0.8) (drill 0.4) (layers F.Cu B.Cu) (net 1))
+  (via (at 301.752 53.086) (size 0.8) (drill 0.4) (layers F.Cu B.Cu) (net 1))
   (segment (start 168.587146 104.851915) (end 170.156343 106.421114) (width 0.29972) (layer B.Cu) (net 6))
   (segment (start 168.19525 104.851914) (end 168.587146 104.851915) (width 0.29972) (layer B.Cu) (net 6))
@@
   (segment (start 151.101399 67.73627) (end 152.310809 66.52686) (width 0.508) (layer F.Cu) (net 13))
   (segment (start 151.101399 70.208801) (end 151.101399 67.73627) (width 0.508) (layer F.Cu) (net 13))
+  (segment (start 12.072246 70.108918) (end 12.072246 69.715754) (width 0.508) (layer F.Cu) (net 13))
   (segment (start 172.505548 102.851917) (end 172.508382 102.854759) (width 0.29972) (layer B.Cu) (net 14))
   (segment (start 168.19525 102.851915) (end 172.505548 102.851917) (width 0.29972) (layer B.Cu) (net 14))

Commit message: DRC III
Switch to usb type-C
Parts:
- added R72: 5.1k, Resistor_SMD:R_0603_1608Metric, B.Cu at (165.1, 42.9)
- added R73: 5.1k, Resistor_SMD:R_0603_1608Metric, B.Cu at (172.2, 42.9)
- USB1: value Molex-0548190589 -> HRO-TYPE-C-31-M-12; footprint MINI:Molex-0548190589 -> Type C:HRO-TYPE-C-31-M-12-jlc
- moved USB1 2.00 mm to (168.6, 30.6), turned to 0 degrees
- moved F1 1.23 mm to (173.0, 45.8)
- moved U3 0.49 mm to (168.6, 44.4)
- turned C12 to 270 degrees
- turned R2 to 270 degrees
Connections:
- C12 pad 1: GND -> Net-(C12-Pad1)
- C12 pad 2: Net-(C12-Pad2) -> GND
- R2 pad 1: GND -> Net-(C12-Pad1)
- R2 pad 2: Net-(C12-Pad2) -> GND
- USB1 pad 2: Net-(USB1-Pad2) -> VBUS
- USB1 pad 3: D+ -> Net-(USB1-Pad3)
- USB1 pad 4: D- -> Net-(R72-Pad2)
- USB1 pad 5: VBUS -> D-
- USB1 pad 6: Net-(C12-Pad2) -> D+
Routing:
- net Net-(C12-Pad1): track 0.00 -> 23.4 mm
- net Net-(C12-Pad2): track 22.6 -> 0.00 mm
- net GND: track 186.3 -> 195.6 mm
- net Net-(R73-Pad2): track 0.00 -> 5.28 mm
- net Net-(R72-Pad2): track 0.00 -> 5.24 mm
- net D-: track 63.6 -> 65.2 mm
- net +5V: track 1745.7 -> 1744.6 mm
- net D+: track 66.3 -> 67.2 mm
- net VBUS: track 17.2 -> 17.8 mm, vias 2 -> 3
Other:
- outline, holes or cut-outs redrawn
- rule pad_to_mask_clearance: 0.05 -> 0

Commit message: DRC IV
Parts:
- USB1: footprint Type C:HRO-TYPE-C-31-M-12-jlc -> edits:HRO-TYPE-C-31-M-12-jlc
- moved G1 49.2 mm to (263.5, 76.2), turned to 0 degrees
- moved Q1 49.2 mm to (146.5, 82.1)
- moved R60 49.2 mm to (269.5, 46.2)
- moved D29 49.2 mm to (254.5, 47.0)
- moved J4 49.2 mm to (152.1, 77.9)
- moved LED1 49.2 mm to (-16.8, 76.6)
- moved MX31 49.2 mm to (135.0, 93.3)
- moved R34 49.2 mm to (138.2, 100.1)
- moved R44 49.2 mm to (190.1, 92.6)
- moved R50 49.2 mm to (222.5, 27.3)
- moved C11 49.2 mm to (154.2, 7.88)
- moved C12 49.2 mm to (157.4, -4.58)
- moved C5 49.2 mm to (152.7, 59.7)
- moved D13 49.2 mm to (113.1, 37.2)
- moved D19 49.2 mm to (170.6, 39.1)
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Routing:
- net IND2: track 213.9 -> 216.9 mm
- net +5V: track 1744.6 -> 1742.1 mm
- net IND3: track 214.7 -> 216.7 mm
- net C5: track 137.5 -> 138.9 mm

Commit message: Checking Datasheet
Parts:
- G1: moved to F.Cu
- moved C7 12.1 mm to (138.7, 52.6), turned to 90 degrees
- moved C10 7.25 mm to (146.9, 3.08)
- moved U2 7.25 mm to (147.1, 5.67)
- moved C11 7.25 mm to (146.9, 8.26)
- moved R1 2.07 mm to (149.1, 46.9), turned to 180 degrees
- moved G1 1.76 mm to (264.3, 77.8)
- moved C13 0.95 mm to (141.4, 65.3), turned to 180 degrees
- moved R3 0.74 mm to (155.7, 57.7)
- moved C4 0.33 mm to (149.7, 50.0)
- moved Y1 0.33 mm to (147.0, 67.1)
- moved C1 0.12 mm to (144.4, 64.1)
Routing:
- net GND: track 195.6 -> 145.1 mm
- net D-: track 65.2 -> 103.9 mm
- net D+: track 67.2 -> 103.9 mm
- net R4: track 241.2 -> 225.8 mm
- net +5V: track 1742.1 -> 1755.0 mm, vias 24 -> 25
- net R3: track 283.8 -> 272.2 mm
- net SWCLK: track 38.8 -> 28.0 mm
- net SWDIO: track 52.3 -> 44.1 mm
- net LED_PWM: track 44.3 -> 37.0 mm
- net VBAT: track 109.2 -> 116.4 mm, vias 6 -> 4
- net IND2: track 216.9 -> 211.3 mm
- net IND1: track 217.7 -> 212.4 mm
- net IND3: track 216.7 -> 211.5 mm
- net R0: track 323.7 -> 328.7 mm, vias 2 -> 3
- net C1: track 229.0 -> 230.1 mm
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
Commit message: DRC Pass
Parts:
- added J1: Conn_01x01_Female, TestPoint:TestPoint_Pad_D1.5mm, B.Cu at (152.0, 94.1)
- J2, J3, J4: value Conn_01x01_Male -> Conn_01x01_Female
- moved C10 28.5 mm to (143.9, 31.4), turned to 270 degrees
- moved U2 26.7 mm to (140.9, 31.6), turned to 90 degrees
- moved C11 24.9 mm to (137.8, 31.4), turned to 90 degrees
- moved J2 18.7 mm to (152.0, 91.6)
- moved J3 13.7 mm to (152.0, 89.0)
- moved J4 8.57 mm to (152.0, 86.5)
- moved U3 2.27 mm to (151.1, 0.70)
- moved F1 2.18 mm to (154.6, 1.78), turned to 90 degrees
- moved R3 1.79 mm to (157.4, 56.9), turned to 0 degrees
- moved R2 1.52 mm to (159.7, -5.97)
- moved C12 1.50 mm to (158.0, -5.97)
- moved C13 1.29 mm to (141.5, 66.6), turned to 270 degrees
- moved C8 1.26 mm to (152.2, 68.0)
- moved R1 1.11 mm to (149.1, 48.0)
- moved Y1 1.02 mm to (148.0, 67.1)
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Connections:
- J3 pad 1: SWDIO -> SWCLK
- J4 pad 1: SWCLK -> VBAT
- U1 pad 11: C14 -> Net-(U1-Pad11)
- U1 pad 12: C7 -> R4
- U1 pad 13: C6 -> R3
- U1 pad 14: C5 -> C6
- U1 pad 15: C4 -> C5
- U1 pad 16: C3 -> C4
- U1 pad 17: C2 -> C3
- U1 pad 18: C1 -> C2
- U1 pad 19: C0 -> C1
- U1 pad 20: R1 -> C0
- U1 pad 21: R3 -> R1
- U1 pad 22: R4 -> C7
- U1 pad 29: R0 -> ENCA
- U1 pad 3: Net-(U1-Pad3) -> C14
- U1 pad 30: ENCA -> ENCB
- U1 pad 31: ENCB -> R0
Routing:
- net R0: track 328.7 -> 292.4 mm
- net SWDIO: track 44.1 -> 61.5 mm
- net R3: track 272.2 -> 259.3 mm
- net SWCLK: track 28.0 -> 39.4 mm
- net R4: track 225.8 -> 214.5 mm
- net C7: track 60.7 -> 49.6 mm
- net C14: track 221.6 -> 213.5 mm, vias 3 -> 1
- net GND: track 145.1 -> 140.2 mm, vias 31 -> 45
- net +5V: track 1755.0 -> 1752.4 mm, vias 25 -> 23
- net Net-(MX6-Pad4): track 13.1 -> 15.2 mm
- net IND3: track 211.5 -> 209.9 mm
- net LED_GND: track 1526.5 -> 1528.0 mm
- net IND1: track 212.4 -> 211.0 mm
- net Net-(C9-Pad1): track 10.8 -> 9.47 mm
- net Net-(MX26-Pad4): track 11.6 -> 12.9 mm
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Other:
- net class Power: via_dia 1.016 -> 0.8; via_drill 0.762 -> 0.4
- board text added: "3.3V"
