File: f103.sch (KiCad schematic (older format))
At the start: 213 parts, among them J1 Conn_01x01_Female, J2 Conn_01x01_Female, J3 Conn_01x01_Female, J4 Conn_01x01_Female, Q1 2N7002, SW1 Rotary_Encoder_Switch, U1 STM32F103CBTx, U2 XC6206P332MR, U3 SRV05-4, Y1 8MHz

Commit message: Finalizing
- Firmware creation begun
- add .step model of PCB
- add gerbers, CPL, BOM
Parts:
- SW1: footprint Rotary_Encoder:RotaryEncoder_Alps_EC11E-Switch_Vertical_H20mm -> edits:RotaryEncoder_Alps_EC11E-Switch_Vertical_H20mm
Connections:
- net ENCA renamed EA
- net ENCB renamed EB
Changed lines of the file:
@@
 	1950 3900 2200 3900
 Connection ~ 2200 3900
-$Comp
-L Device:Rotary_Encoder_Switch SW1
-U 1 1 60062B88
-P 950 1800
-F 0 "SW1" V 1400 2050 50  0000 R CNN
-F 1 "Rotary_Encoder_Switch" V 1300 2150 20  0000 R CNN
-F 2 "Rotary_Encoder:RotaryEncoder_Alps_EC11E-Switch_Vertical_H20mm" H 800 1960 50  0001 C CNN
-F 3 "~" H 950 2060 50  0001 C CNN
-	1    950  1800
-	0    -1   -1   0
-$EndComp
-Wire Wire Line
-	1050 1500 1500 1500
-Connection ~ 1500 1500
-Wire Wire Line
-	1500 1500 1500 1350
-Wire Wire Line
-	1300 1950 1200 1950
-Wire Wire Line
-	1200 1950 1200 1550
-Wire Wire Line
-	1200 1550 850  1550
-Wire Wire Line
-	850  1550 850  1500
-$Comp
-L power:GND #PWR0133
-U 1 1 600CA7BC
-P 950 2350
-F 0 "#PWR0133" H 950 2100 50  0001 C CNN
-F 1 "GND" H 955 2177 50  0000 C CNN
-F 2 "" H 950 2350 50  0001 C CNN
-F 3 "" H 950 2350 50  0001 C CNN
-	1    950  2350
-	1    0    0    -1
-$EndComp
-Text GLabel 850  2100 3    50   Input ~ 0
-ENCA
-Text GLabel 1050 2100 3    50   Input ~ 0
-ENCB
-Text GLabel 15300 4700 2    50   Input ~ 0
-ENCB
-Text GLabel 15300 4600 2    50   Input ~ 0
-ENCA
 Wire Wire Line
 	15300 5000 15650 5000
@@
 	2400 3600 2400 4500
 Wire Wire Line
-	1500 1500 1500 1750
-Wire Wire Line
 	3050 1350 3050 1750
 Wire Wire Line
@@
 Wire Wire Line
 	1500 1750 1500 2650
-Connection ~ 1300 1950
 Connection ~ 1450 1800
 Wire Wire Line
@@
 Connection ~ 950  8050
 Connection ~ 950  8350
-Wire Wire Line
-	950  2350 950  2100
 $Comp
 L power:+3.3V #PWR0132
@@
 Wire Wire Line
 	14000 8000 14450 8000
+Wire Wire Line
+	1500 1350 1500 1600
+$Comp
+L Device:Rotary_Encoder_Switch SW1
+U 1 1 6048E041
+P -450 1800
+F 0 "SW1" V -404 1570 50  0000 R CNN
+F 1 "Rotary_Encoder_Switch" V -495 1570 50  0000 R CNN
+F 2 "edits:RotaryEncoder_Alps_EC11E-Switch_Vertical_H20mm" H -600 1960 50  0001 C CNN
+F 3 "~" H -450 2060 50  0001 C CNN
+	1    -450 1800
+	0    -1   -1   0
+$EndComp
+$Comp
+L power:GND #PWR0129
+U 1 1 604914B2
+P -450 2100
+F 0 "#PWR0129" H -450 1850 50  0001 C CNN
+F 1 "GND" H -445 1927 50  0000 C CNN
+F 2 "" H -450 2100 50  0001 C CNN
+F 3 "" H -450 2100 50  0001 C CNN
+	1    -450 2100
+	1    0    0    -1
+$EndComp
+Text GLabel -550 2100 0    50   Input ~ 0
+EA
+Text GLabel -350 2100 2    50   Input ~ 0
+EB
+Wire Wire Line
+	1300 1950 -100 1950
+Wire Wire Line
+	-100 1950 -100 2350
+Wire Wire Line
+	-100 2350 -850 2350
+Wire Wire Line
+	-850 2350 -850 1500
+Wire Wire Line
+	-850 1500 -550 1500
+Connection ~ 1300 1950
+Wire Wire Line
+	1500 1600 -150 1600
+Wire Wire Line
+	-150 1600 -150 1500
+Wire Wire Line
+	-150 1500 -350 1500
+Connection ~ 1500 1600
+Wire Wire Line
+	1500 1600 1500 1750
+Text GLabel 15300 4700 2    50   Input ~ 0
+EB
+Text GLabel 15300 4600 2    50   Input ~ 0
+EA
 $EndSCHEMATC

Commit message: overhaul: see description
- remapped backlighting to A9
- remapped encoder pad B to B12
- updated ground fills
- added 02 silkscreen
- write firmware
- add compiled binary file
- begin acrylic case
- update gerbers and component placement files
- update readme images
Parts:
- added G2, G3: zero, Graphics:02, symbol Mechanical:MountingHole
Connections:
- net EB: now also U1.25 (PB12); no longer U1.30 (PA9)
- net LED_PWM: now also U1.30 (PA9); no longer U1.25 (PB12)
Other:
- moved on the sheet: C1, C13, C2, C3, C4, C5, C6, C7, C8, C9, D1, D10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

Commit message: ordered prototypes
Parts:
- G2, G3: footprint Graphics:02 -> Graphics:0222
Changed lines of the file:
@@
 F 0 "G2" H 8950 7546 50  0000 L CNN
 F 1 "zero" H 8950 7455 50  0000 L CNN
-F 2 "Graphics:02" H 8850 7500 50  0001 C CNN
+F 2 "Graphics:0222" H 8850 7500 50  0001 C CNN
 F 3 "~" H 8850 7500 50  0001 C CNN
 	1    8850 7500
@@
 F 0 "G3" H 9350 7546 50  0000 L CNN
 F 1 "zero" H 9350 7455 50  0000 L CNN
-F 2 "Graphics:02" H 9250 7500 50  0001 C CNN
+F 2 "Graphics:0222" H 9250 7500 50  0001 C CNN
 F 3 "~" H 9250 7500 50  0001 C CNN
 	1    9250 7500
